File: Hardware/STM32H7_Car/STM32H7_Car.kicad_pcb (KiCad board)
At the start: 2 copper layers, 1 part

Commit message: 归档硬件设计与项目参考资料快照
Parts:
- added C1: 22u, Capacitor_SMD:C_0805_2012Metric, F.Cu at (112.4, 120.4)
- added C10: 22p, Capacitor_SMD:C_0603_1608Metric, F.Cu at (92.2, 117.5)
- added C11: 4.7n, Capacitor_SMD:C_0603_1608Metric, F.Cu at (95.8, 114.4)
- added C12: 0.1u, Capacitor_SMD:C_0603_1608Metric, F.Cu at (83.2, 115.4)
- added C13: 22u, Capacitor_SMD:C_0805_2012Metric, F.Cu at (80.1, 116.4)
- added C14: 22u, Capacitor_SMD:C_0805_2012Metric, F.Cu at (78.1, 116.4)
- added C15: 1u, Capacitor_SMD:C_0603_1608Metric, F.Cu at (95.8, 115.9)
- added C16: 1u, Capacitor_SMD:C_0603_1608Metric, F.Cu at (122.0, 113.8)
- added C17: 1u, Capacitor_SMD:C_0603_1608Metric, F.Cu at (73.3, 103.5)
- added C18: 1u, Capacitor_SMD:C_0603_1608Metric, F.Cu at (73.3, 106.0)
- added C19: 0.1u, Capacitor_SMD:C_0603_1608Metric, F.Cu at (109.2, 128.4)
- added C2: 0.1u, Capacitor_SMD:C_0603_1608Metric, F.Cu at (112.4, 118.6)
- added C3: 22p, Capacitor_SMD:C_0603_1608Metric, F.Cu at (122.0, 115.3)
- added C4: 10n, Capacitor_SMD:C_0603_1608Metric, F.Cu at (122.0, 112.3)
- added C5: 0.1u, Capacitor_SMD:C_0603_1608Metric, F.Cu at (109.7, 115.7)
- added C6: 22u, Capacitor_SMD:C_0805_2012Metric, F.Cu at (106.7, 116.7)
- added C7: 22u, Capacitor_SMD:C_0805_2012Metric, F.Cu at (104.7, 116.7)
- added C8: 10u, Capacitor_SMD:C_0805_2012Metric, F.Cu at (85.6, 119.3)
- added C9: 0.1u, Capacitor_SMD:C_0603_1608Metric, F.Cu at (85.6, 117.5)
- added J1: L_MOTOR, Connector_PinHeader_2.54mm:PinHeader_1x03_P2.54mm_Vertical, F.Cu at (60.0, 109.4)
- added J10: USART1, Connector_PinHeader_2.54mm:PinHeader_1x04_P2.54mm_Vertical, F.Cu at (82.5, 91.0)
- added J11: DL1B, Connector_PinHeader_2.54mm:PinHeader_1x05_P2.54mm_Vertical, F.Cu at (94.8, 43.0)
- added J12: M_MOTOR, Connector_PinHeader_2.54mm:PinHeader_1x03_P2.54mm_Vertical, F.Cu at (54.9, 102.5)
- added J13: USART2, Connector_PinHeader_2.54mm:PinHeader_1x04_P2.54mm_Vertical, F.Cu at (109.4, 91.0)
- added J14: SPI_NC, Connector_PinHeader_2.54mm:PinHeader_1x08_P2.54mm_Vertical, F.Cu at (124.0, 21.4)
- added J15: XT30PW-M, Connector_AMASS:AMASS_XT30PW-M_1x02_P2.50mm_Horizontal, F.Cu at (136.1, 140.9)
- added J16: 5V, Connector_PinHeader_2.54mm:PinHeader_1x02_P2.54mm_Vertical, F.Cu at (102.7, 140.6)
- added J17: 5V, Connector_PinHeader_2.54mm:PinHeader_1x02_P2.54mm_Vertical, F.Cu at (111.8, 140.6)
- added J18: 5V, Connector_PinHeader_2.54mm:PinHeader_1x02_P2.54mm_Vertical, F.Cu at (121.2, 140.6)
- added J2: R_MOTOR, Connector_PinHeader_2.54mm:PinHeader_1x03_P2.54mm_Vertical, F.Cu at (141.0, 108.5)
- added J3: L_ENC, Connector_PinHeader_1.27mm:PinHeader_1x04_P1.27mm_Vertical, F.Cu at (61.5, 122.1)
- added J3A: FPC-SMD_4P-P1.00_JS_AFA01-S04FCA-00, Library:FPC-SMD_4P-P1.00_JS_AFA01-S04FCA-00, F.Cu at (57.2, 123.9)
- added J4: R_ENC, Connector_PinHeader_1.27mm:PinHeader_1x04_P1.27mm_Vertical, F.Cu at (137.4, 127.4)
- added J4A: FPC-SMD_4P-P1.00_JS_AFA01-S04FCA-00, Library:FPC-SMD_4P-P1.00_JS_AFA01-S04FCA-00, F.Cu at (141.9, 125.4)
- added J5: L_ADC, Connector_PinHeader_2.54mm:PinHeader_1x07_P2.54mm_Vertical, F.Cu at (74.1, 91.0)
- added J5A: FPC-SMD_XUNPU_FPC-1.0FX-7PWCR-H20, Library:FPC-SMD_XUNPU_FPC-1.0FX-7PWCR-H20, F.Cu at (59.5, 81.9)
- added J6: IR_ADC, Connector_PinHeader_2.54mm:PinHeader_1x07_P2.54mm_Vertical, F.Cu at (141.5, 91.0)
- added J6A: FPC-SMD_XUNPU_FPC-1.0FX-7PWCR-H20, Library:FPC-SMD_XUNPU_FPC-1.0FX-7PWCR-H20, F.Cu at (141.0, 81.4)
- added J7: IMU, Connector_PinHeader_2.54mm:PinHeader_1x06_P2.54mm_Vertical, F.Cu at (68.4, 140.7)
- added J7A: FPC-SMD_6P-P1.00_AFA01-S06, Library:FPC-SMD_6P-P1.00_AFA01-S06, F.Cu at (58.3, 140.4)
- added J8: OLED, Connector_PinHeader_2.54mm:PinHeader_1x08_P2.54mm_Vertical, F.Cu at (47.8, 159.7)
- added J9: WIFI, Connector_PinHeader_2.54mm:PinHeader_2x04_P2.54mm_Vertical, F.Cu at (26.8, 80.5)
- added L1: 3.3u, Library:L_Molded_5x5mm_FEXL0530A_ZD0520, F.Cu at (108.2, 111.8)
- added L2: 2.2u, Library:L_Molded_5x5mm_FEXL0530A_ZD0520, F.Cu at (81.2, 111.3)
- added R1: 10k, Resistor_SMD:R_0603_1608Metric, F.Cu at (117.7, 118.6)
- added R2: 124k, Resistor_SMD:R_0603_1608Metric, F.Cu at (122.0, 116.8)
- added R3: 22.1k, Resistor_SMD:R_0603_1608Metric, F.Cu at (122.0, 118.3)
- added R4: 73.2k, Resistor_SMD:R_0603_1608Metric, F.Cu at (92.2, 119.0)
- added R5: 22.1k, Resistor_SMD:R_0603_1608Metric, F.Cu at (95.8, 117.4)
- added R6: 10k, Resistor_SMD:R_0603_1608Metric, F.Cu at (95.8, 111.4)
- added R7: 100k, Resistor_SMD:R_0603_1608Metric, F.Cu at (95.8, 112.9)
- added R8: 100k, Resistor_SMD:R_0603_1608Metric, F.Cu at (106.2, 128.4)
- added R9: 27k, Resistor_SMD:R_0603_1608Metric, F.Cu at (107.7, 128.4)
- added U1: TPS54627DDAR, Library:TI_DDA0008A_SO-PowerPAD-8, F.Cu at (116.0, 114.3)
- added U2: TPS54325PWPR, Library:TI_PWP0014A_HTSSOP-14-EP, F.Cu at (89.4, 113.5)
- added U3: TPS7A2033PDBVR, Library:SOT-23-5, F.Cu at (77.8, 105.0)
- added U4: ESP32-S3-DevKitM-1, Library:ESP32-S3-DevKitM-1, F.Cu at (99.9, 74.0)
- moved 1 21.1 mm to (100.0, 115.5), turned to 90 degrees
Connections:
- 1 pad 1: +3.3V -> unconnected-(1A-3V3-Pad1)
- 1 pad 42: +3.3V -> unconnected-(1A-3V3-Pad42)
- 1 pad 9: unconnected-(1A-NRST-Pad9) -> /stm32_RST
Other:
- board outline added: 98 x 85 mm
